Commit message: add FMB benchmark usd files

File: xarm_rl/models/FMB/mount/side_mount.urdf (robot description, URDF)
Before this commit: robot side_mount, 1 links, 0 joints
Links:
- link side_mount: geometry collision mesh filename=./side_mount.stl scale=0.001 0.001 0.001; visual mesh filename=./side_mount.stl scale=0.001 0.001 0.001

File: xarm_rl/models/FMB/mount/wrist_mount.urdf (robot description, URDF)
Before this commit: robot wrist_mount, 1 links, 0 joints
Links:
- link wrist_mount: geometry collision mesh filename=./wrist_mount.stl scale=0.001 0.001 0.001; visual mesh filename=./wrist_mount.stl scale=0.001 0.001 0.001
