Commit message: fix path

File: xarm_rl/models/urdf/fmb/momo/assembly1/base.urdf (robot description, URDF)
Before this commit: robot base, 1 links, 0 joints
Links:
- link base: geometry collision mesh filename=./meshes/base.stl scale=0.001 0.001 0.001; visual mesh filename=./meshes/base.stl scale=0.001 0.001 0.001

File: xarm_rl/models/urdf/fmb/momo/assembly1/block1.urdf (robot description, URDF)
Before this commit: robot block1, 1 links, 0 joints
Links:
- link block1: geometry collision mesh filename=./meshes/block1.stl scale=0.001 0.001 0.001; visual mesh filename=./meshes/block1.stl scale=0.001 0.001 0.001

File: xarm_rl/models/urdf/fmb/momo/assembly1/block2.urdf (robot description, URDF)
Before this commit: robot block2, 1 links, 0 joints
Links:
- link block2: geometry collision mesh filename=./meshes/block2.stl scale=0.001 0.001 0.001; visual mesh filename=./meshes/block2.stl scale=0.001 0.001 0.001

File: xarm_rl/models/urdf/fmb/momo/assembly1/block3.urdf (robot description, URDF)
Before this commit: robot block3, 1 links, 0 joints
Links:
- link block3: geometry collision mesh filename=./meshes/block3.stl scale=0.001 0.001 0.001; visual mesh filename=./meshes/block3.stl scale=0.001 0.001 0.001

File: xarm_rl/models/urdf/fmb/momo/assembly1/block4.urdf (robot description, URDF)
Before this commit: robot block4, 1 links, 0 joints
Links:
- link block4: geometry collision mesh filename=./meshes/block4.stl scale=0.001 0.001 0.001; visual mesh filename=./meshes/block4.stl scale=0.001 0.001 0.001
