Commit message: :tada: fetch & stack

File: xarm_tamp/tampkit/models/urdf/fmb_momo/Assembly1/urdf/Board1_Base.urdf (robot description, URDF)
Before this commit: robot board1_base, 1 links, 0 joints
Links:
- removed link board1_base
- added link base; collision mesh filename=../meshes/base.stl; visual mesh filename=../meshes/base.stl

File: xarm_tamp/tampkit/models/urdf/fmb_momo/Assembly1/urdf/Board1_Block1.urdf (robot description, URDF)
Before this commit: robot board1_block1, 1 links, 0 joints
Links:
- removed link board1_block1
- added link block1; collision mesh filename=../meshes/block1.stl; visual mesh filename=../meshes/block1.stl

File: xarm_tamp/tampkit/models/urdf/fmb_momo/Assembly1/urdf/Board1_Block2.urdf (robot description, URDF)
Before this commit: robot board1_block2, 1 links, 0 joints
Links:
- removed link board1_block2
- added link block2; collision mesh filename=../meshes/block2.stl; visual mesh filename=../meshes/block2.stl

File: xarm_tamp/tampkit/models/urdf/fmb_momo/Assembly1/urdf/Board1_Block3.urdf (robot description, URDF)
Before this commit: robot board1_block3, 1 links, 0 joints
Links:
- removed link board1_block3
- added link block3; collision mesh filename=../meshes/block3.stl; visual mesh filename=../meshes/block3.stl

File: xarm_tamp/tampkit/models/urdf/fmb_momo/Assembly1/urdf/Board1_Block4.urdf (robot description, URDF)
Before this commit: robot board1_block4, 1 links, 0 joints
Links:
- removed link board1_block4
- added link block4; collision mesh filename=../meshes/block4.stl; visual mesh filename=../meshes/block4.stl
